File: Hardware/RocketBrain.sch (KiCad schematic (older format))
At the start: 0 parts

Commit message: Update schematic and routing
Changed lines of the file:
@@
 F4 "~CS_SD" O R 6900 3300 50
 F5 "~CS_flash" O R 6900 3400 50
-F6 "pyro" O R 6900 3050 50
+F6 "pyro1" O R 6900 3050 50
 F7 "~RESET_LoRa" O L 5200 3175 50
 F8 "~CS_LoRa" O L 5200 3300 50
 F9 "INT_6050" O L 5200 3450 50
+F10 "pyro2" O R 6900 3150 50
 $EndSheet
 Wire Wire Line
@@
 F0 "Pyro" 50
 F1 "pyro.sch" 50
-F2 "pyro" I R 6900 2325 50
+F2 "pyro1" I R 6900 2325 50
+F3 "pyro2" I R 6900 2200 50
 $EndSheet
 Wire Wire Line
@@
 Wire Wire Line
 	5200 3450 4425 3450
+Wire Wire Line
+	6900 3150 7100 3150
+Wire Wire Line
+	7100 3150 7100 2200
+Wire Wire Line
+	7100 2200 6900 2200
 $EndSCHEMATC
