File: Hardware/navigation.sch (KiCad schematic (older format))
At the start: 19 parts, among them U2 LSM9DS1, U3 MPU-6050, U6 BMP280

Commit message: Change regulator diode footprint, update routing
Parts:
- U2: MANUFACTURER (none) -> STMicroelectronics; Manufacturer_Part_Number (none) -> LSM9DS1
- U3: MANUFACTURER (none) -> TDK InvenSense; Manufacturer_Part_Number (none) -> MPU-6050
- U6: MANUFACTURER (none) -> Bosch Sensortec; Manufacturer_Part_Number (none) -> BMP280
Changed lines of the file:
@@
 F 2 "Sensor_Motion:InvenSense_QFN-24_4x4mm_P0.5mm" H 3750 1600 50  0001 C CNN
 F 3 "https://store.invensense.com/datasheets/invensense/MPU-6050_DataSheet_V3%204.pdf" H 3750 2250 50  0001 C CNN
+F 4 "TDK InvenSense" H 3750 2400 50  0001 C CNN "MANUFACTURER"
+F 5 "MPU-6050" H 3750 2400 50  0001 C CNN "Manufacturer_Part_Number"
 	1    3750 2400
 	1    0    0    -1
@@
 F 2 "Package_LGA:LGA-24L_3x3.5mm_P0.43mm" H 5225 6100 50  0001 C CNN
 F 3 "http://www.st.com/content/ccc/resource/technical/document/datasheet/1e/3f/2a/d6/25/eb/48/46/DM00103319.pdf/files/DM00103319.pdf/jcr:content/translations/en.DM00103319.pdf" H 3725 5450 50  0001 C CNN
+F 4 "STMicroelectronics" H 3725 5350 50  0001 C CNN "MANUFACTURER"
+F 5 "LSM9DS1" H 3725 5350 50  0001 C CNN "Manufacturer_Part_Number"
 	1    3725 5350
 	1    0    0    -1
@@
 F 2 "Package_LGA:Bosch_LGA-8_2x2.5mm_P0.65mm_ClockwisePinNumbering" H 7550 3575 50  0001 C CNN
 F 3 "https://ae-bst.resource.bosch.com/media/_tech/media/datasheets/BST-BMP280-DS001.pdf" H 7550 4275 50  0001 C CNN
+F 4 "Bosch Sensortec" H 7550 4275 50  0001 C CNN "MANUFACTURER"
+F 5 "BMP280" H 7550 4275 50  0001 C CNN "Manufacturer_Part_Number"
 	1    7550 4275
 	1    0    0    -1
